File: rfmodules.sch (KiCad schematic (older format))
At the start: 8 parts, among them U6 LP38693SD-3.3

Commit message: Small changes
Parts:
- renumbered C19 to C29, C20 to C30, C21 to C31, C22 to C32, C23 to C33
Changed lines of the file:
@@
 $EndDescr
 $Comp
-L power:GND #PWR025
+L power:GND #PWR028
 U 1 1 5C7BA0F1
 P 4100 3650
-F 0 "#PWR025" H 4100 3400 50  0001 C CNN
+F 0 "#PWR028" H 4100 3400 50  0001 C CNN
 F 1 "GND" H 4105 3477 50  0000 C CNN
 F 2 "" H 4100 3650 50  0001 C CNN
@@
 $EndComp
 $Comp
-L power:GND #PWR027
+L power:GND #PWR030
 U 1 1 5C7BA229
 P 4075 5925
-F 0 "#PWR027" H 4075 5675 50  0001 C CNN
+F 0 "#PWR030" H 4075 5675 50  0001 C CNN
 F 1 "GND" H 4080 5752 50  0000 C CNN
 F 2 "" H 4075 5925 50  0001 C CNN
@@
 $EndComp
 $Comp
-L Device:C C21
+L Device:C C31
 U 1 1 5C7BA5D5
 P 3125 1975
-F 0 "C21" H 3240 2021 50  0000 L CNN
+F 0 "C31" H 3240 2021 50  0000 L CNN
 F 1 "1uF" H 3240 1930 50  0000 L CNN
 F 2 "" H 3163 1825 50  0001 C CNN
@@
 $EndComp
 $Comp
-L Device:C C20
+L Device:C C30
 U 1 1 5C7BA627
 P 1675 1975
-F 0 "C20" H 1790 2021 50  0000 L CNN
+F 0 "C30" H 1790 2021 50  0000 L CNN
 F 1 "1uF" H 1790 1930 50  0000 L CNN
 F 2 "" H 1713 1825 50  0001 C CNN
@@
 Connection ~ 2500 2250
 $Comp
-L power:GND #PWR024
+L power:GND #PWR027
 U 1 1 5C7BB12C
 P 2500 2300
-F 0 "#PWR024" H 2500 2050 50  0001 C CNN
+F 0 "#PWR027" H 2500 2050 50  0001 C CNN
 F 1 "GND" H 2505 2127 50  0000 C CNN
 F 2 "" H 2500 2300 50  0001 C CNN
@@
 Connection ~ 1675 2250
 $Comp
-L Device:C C19
+L Device:C C29
 U 1 1 5C7CD227
 P 4375 1825
-F 0 "C19" V 4123 1825 50  0000 C CNN
+F 0 "C29" V 4123 1825 50  0000 C CNN
 F 1 "100nF" V 4214 1825 50  0000 C CNN
 F 2 "" H 4413 1675 50  0001 C CNN
@@
 $EndComp
 $Comp
-L Device:C C23
+L Device:C C33
 U 1 1 5C7CD2B2
 P 4375 4350
-F 0 "C23" V 4123 4350 50  0000 C CNN
+F 0 "C33" V 4123 4350 50  0000 C CNN
 F 1 "100nF" V 4214 4350 50  0000 C CNN
 F 2 "" H 4413 4200 50  0001 C CNN
@@
 $EndComp
 $Comp
-L power:GND #PWR022
+L power:GND #PWR025
 U 1 1 5C7CD32E
 P 4600 1875
-F 0 "#PWR022" H 4600 1625 50  0001 C CNN
+F 0 "#PWR025" H 4600 1625 50  0001 C CNN
 F 1 "GND" H 4605 1702 50  0000 C CNN
 F 2 "" H 4600 1875 50  0001 C CNN
@@
 $EndComp
 $Comp
-L power:GND #PWR026
+L power:GND #PWR029
 U 1 1 5C7CD35E
 P 4600 4425
-F 0 "#PWR026" H 4600 4175 50  0001 C CNN
+F 0 "#PWR029" H 4600 4175 50  0001 C CNN
 F 1 "GND" H 4605 4252 50  0000 C CNN
 F 2 "" H 4600 4425 50  0001 C CNN
@@
 	4075 4350 4075 4725
 $Comp
-L Device:CP C22
+L Device:CP C32
 U 1 1 5C8A056F
 P 3725 2025
-F 0 "C22" H 3843 2071 50  0000 L CNN
+F 0 "C32" H 3843 2071 50  0000 L CNN
 F 1 "100uF" H 3843 1980 50  0000 L CNN
 F 2 "" H 3763 1875 50  0001 C CNN
@@
 $EndComp
 $Comp
-L power:GND #PWR023
+L power:GND #PWR026
 U 1 1 5C8A05FA
 P 3725 2225
-F 0 "#PWR023" H 3725 1975 50  0001 C CNN
+F 0 "#PWR026" H 3725 1975 50  0001 C CNN
 F 1 "GND" H 3575 2150 50  0000 C CNN
 F 2 "" H 3725 2225 50  0001 C CNN

Commit message: Final changes in schema
Parts:
- C31: renamed from C32; value 100uF -> 10uF
- renumbered C29 to C28, C30 to C29, C31 to C30, C33 to C32
Changed lines of the file:
@@
 encoding utf-8
 Sheet 3 3
-Title ""
-Date ""
-Rev ""
-Comp ""
-Comment1 ""
+Title "SX1280 based RC receiver"
+Date "2019-02-25"
+Rev "1"
+Comp "bodrico.com"
+Comment1 "Designed by bodri@bodrico.com"
 Comment2 ""
 Comment3 ""
@@
 $EndComp
 $Comp
-L Device:C C31
+L Device:C C30
 U 1 1 5C7BA5D5
 P 3125 1975
-F 0 "C31" H 3240 2021 50  0000 L CNN
+F 0 "C30" H 3240 2021 50  0000 L CNN
 F 1 "1uF" H 3240 1930 50  0000 L CNN
 F 2 "" H 3163 1825 50  0001 C CNN
@@
 $EndComp
 $Comp
-L Device:C C30
+L Device:C C29
 U 1 1 5C7BA627
 P 1675 1975
-F 0 "C30" H 1790 2021 50  0000 L CNN
+F 0 "C29" H 1790 2021 50  0000 L CNN
 F 1 "1uF" H 1790 1930 50  0000 L CNN
 F 2 "" H 1713 1825 50  0001 C CNN
@@
 Connection ~ 1675 2250
 $Comp
-L Device:C C29
+L Device:C C28
 U 1 1 5C7CD227
 P 4375 1825
-F 0 "C29" V 4123 1825 50  0000 C CNN
+F 0 "C28" V 4123 1825 50  0000 C CNN
 F 1 "100nF" V 4214 1825 50  0000 C CNN
 F 2 "" H 4413 1675 50  0001 C CNN
@@
 $EndComp
 $Comp
-L Device:C C33
+L Device:C C32
 U 1 1 5C7CD2B2
 P 4375 4350
-F 0 "C33" V 4123 4350 50  0000 C CNN
+F 0 "C32" V 4123 4350 50  0000 C CNN
 F 1 "100nF" V 4214 4350 50  0000 C CNN
 F 2 "" H 4413 4200 50  0001 C CNN
@@
 	4075 4350 4075 4725
 $Comp
-L Device:CP C32
+L Device:CP C31
 U 1 1 5C8A056F
 P 3725 2025
-F 0 "C32" H 3843 2071 50  0000 L CNN
-F 1 "100uF" H 3843 1980 50  0000 L CNN
+F 0 "C31" H 3843 2071 50  0000 L CNN
+F 1 "10uF" H 3843 1980 50  0000 L CNN
 F 2 "" H 3763 1875 50  0001 C CNN
 F 3 "~" H 3725 2025 50  0001 C CNN

Commit message: Add some footprints
Parts:
- A1, A2: footprint (none) -> miscellaneous:E28-2G4M20S
- C28, C29, C30, C32: footprint (none) -> Capacitor_SMD:C_0402_1005Metric
- C31: footprint (none) -> Capacitor_Tantalum_SMD:CP_EIA-3216-18_Kemet-A
- U6: footprint (none) -> miscellaneous:WSON-6_3x3mm_Pitch0.95mm
Changed lines of the file:
@@
 EESchema Schematic File Version 4
+LIBS:RcReceiver-cache
 EELAYER 26 0
 EELAYER END
@@
 F 0 "U6" H 2500 2290 50  0000 C CNN
 F 1 "LP38693SD-3.3" H 2500 2199 50  0000 C CNN
-F 2 "" H 2500 1925 50  0001 C CNN
+F 2 "miscellaneous:WSON-6_3x3mm_Pitch0.95mm" H 2500 1925 50  0001 C CNN
 F 3 "http://www.ti.com/lit/ds/snvs321o/snvs321o.pdf" H 2500 1925 50  0001 C CNN
 	1    2500 1925
@@
 F 0 "C30" H 3240 2021 50  0000 L CNN
 F 1 "1uF" H 3240 1930 50  0000 L CNN
-F 2 "" H 3163 1825 50  0001 C CNN
+F 2 "Capacitor_SMD:C_0402_1005Metric" H 3163 1825 50  0001 C CNN
 F 3 "~" H 3125 1975 50  0001 C CNN
 	1    3125 1975
@@
 F 0 "C29" H 1790 2021 50  0000 L CNN
 F 1 "1uF" H 1790 1930 50  0000 L CNN
-F 2 "" H 1713 1825 50  0001 C CNN
+F 2 "Capacitor_SMD:C_0402_1005Metric" H 1713 1825 50  0001 C CNN
 F 3 "~" H 1675 1975 50  0001 C CNN
 	1    1675 1975
@@
 F 0 "C28" V 4123 1825 50  0000 C CNN
 F 1 "100nF" V 4214 1825 50  0000 C CNN
-F 2 "" H 4413 1675 50  0001 C CNN
+F 2 "Capacitor_SMD:C_0402_1005Metric" H 4413 1675 50  0001 C CNN
 F 3 "~" H 4375 1825 50  0001 C CNN
 	1    4375 1825
@@
 F 0 "C32" V 4123 4350 50  0000 C CNN
 F 1 "100nF" V 4214 4350 50  0000 C CNN
-F 2 "" H 4413 4200 50  0001 C CNN
+F 2 "Capacitor_SMD:C_0402_1005Metric" H 4413 4200 50  0001 C CNN
 F 3 "~" H 4375 4350 50  0001 C CNN
 	1    4375 4350
@@
 F 0 "C31" H 3843 2071 50  0000 L CNN
 F 1 "10uF" H 3843 1980 50  0000 L CNN
-F 2 "" H 3763 1875 50  0001 C CNN
+F 2 "Capacitor_Tantalum_SMD:CP_EIA-3216-18_Kemet-A" H 3763 1875 50  0001 C CNN
 F 3 "~" H 3725 2025 50  0001 C CNN
 	1    3725 2025
@@
 F 0 "A2" H 3675 5775 50  0000 C CNN
 F 1 "E28-2G4M20S" H 4375 5775 50  0000 C CNN
-F 2 "" H 3825 5375 50  0001 C CNN
+F 2 "miscellaneous:E28-2G4M20S" H 3825 5375 50  0001 C CNN
 F 3 "http://www.ebyte.com/en/downpdf.aspx?id=286" H 5225 4725 50  0001 C CNN
 	1    4075 5275
@@
 F 0 "A1" H 3700 3500 50  0000 C CNN
 F 1 "E28-2G4M20S" H 4400 3500 50  0000 C CNN
-F 2 "" H 3850 3100 50  0001 C CNN
+F 2 "miscellaneous:E28-2G4M20S" H 3850 3100 50  0001 C CNN
 F 3 "http://www.ebyte.com/en/downpdf.aspx?id=286" H 5250 2450 50  0001 C CNN
 	1    4100 3000

Commit message: Create PCB
Changed lines of the file:
@@
 Wire Wire Line
 	4075 5900 4125 5900
+Text Label 1675 1825 2    50   ~ 0
+VCC
 $EndSCHEMATC
