File: RcReceiver.kicad_pcb (KiCad board)
At the start: 4 copper layers, 50 x 29.5 mm, 73 parts, among them J1 VBAT, J10 Servo3, J11 Servo4, J12 Servo5, J13 CAN, J14 Servo6, J15 Servo7, J16 Servo8, J17 GND for the Servo connectors, J2 SWD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

Commit message: More routing
Parts:
- moved C14 0.08 mm to (172.3, 60.0)
Routing:
- net GND: track 31.9 -> 280.4 mm, vias 0 -> 31
- net /VCCCPU: track 47.0 -> 165.7 mm, vias 0 -> 9
- net IN: track 0.00 -> 76.4 mm, vias 0 -> 13
- net /RF modules/VCCRF: track 8.42 -> 75.3 mm, vias 0 -> 3
- net /RF1MISO: track 0.00 -> 40.2 mm, vias 0 -> 1
- net /RF1RXEN: track 0.00 -> 26.9 mm, vias 0 -> 1
- net /RF2CLK: track 0.00 -> 16.6 mm, vias 0 -> 1
- net /RF2NSS: track 0.00 -> 15.7 mm, vias 0 -> 1
- net /RF2TXEN: track 0.00 -> 14.2 mm, vias 0 -> 1
- net /RF1TXEN: track 0.00 -> 13.4 mm, vias 0 -> 1
- net /RF2NRESET: track 0.00 -> 13.0 mm, vias 0 -> 1
- net /RF1IRQ: track 0.00 -> 12.0 mm, vias 0 -> 1
- net /RF1BUSY: track 0.00 -> 11.9 mm, vias 0 -> 1
- net /RF1NRESET: track 0.00 -> 11.2 mm, vias 0 -> 1
- net /RF2BUSY: track 0.00 -> 10.3 mm, vias 0 -> 1
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Other:
- net class IN: via_dia 1.016 -> 0.6858; via_drill 0.6 -> 0.3302
- net class VCC: via_dia 1.016 -> 0.6858; via_drill 0.6 -> 0.3302

Commit message: More routing
Parts:
- removed J3: I2C, Connector_JST:JST_SH_BM05B-SRSS-TB_1x05-1MP_P1.00mm_Vertical
- removed J7: SPI3, Connector_JST:JST_SH_BM07B-SRSS-TB_1x07-1MP_P1.00mm_Vertical
Routing:
- net /RF1NSS: track 0.00 -> 48.6 mm, vias 0 -> 1
- net /RF1MOSI: track 0.00 -> 45.4 mm, vias 0 -> 4
- net /TX1: track 0.00 -> 44.2 mm, vias 0 -> 2
- net /Connectors/PWM6: track 0.00 -> 43.6 mm, vias 0 -> 3
- net /Connectors/PWM7: track 0.00 -> 41.8 mm, vias 0 -> 2
- net /Connectors/PWM8: track 0.00 -> 38.9 mm, vias 0 -> 2
- net /Connectors/PWM5: track 0.00 -> 37.4 mm, vias 0 -> 3
- net /SWDIO: track 0.00 -> 35.6 mm, vias 0 -> 2
- net /SWCLK: track 0.00 -> 27.4 mm, vias 0 -> 2
- net /NRST: track 0.00 -> 26.2 mm, vias 0 -> 3
- net /Connectors/VCCOUT: track 19.8 -> 45.8 mm, vias 2 -> 4
- net /RX1: track 0.00 -> 25.3 mm, vias 0 -> 2
- net /RF2MISO: track 0.00 -> 20.3 mm, vias 0 -> 2
- net /RFPOWEREN: track 0.00 -> 20.0 mm, vias 0 -> 2
- net /PWMOE: track 0.00 -> 19.1 mm, vias 0 -> 2
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Other:
- board text removed: "I2C"
- board text removed: "SPI3"

Commit message: More routing
Routing:
- net /PWM3: track 2.59 -> 55.9 mm, vias 1 -> 2
- net /RF1CLK: track 0.00 -> 45.8 mm, vias 0 -> 3
- net /PWM4: track 5.18 -> 50.8 mm, vias 1 -> 2
- net /PWM1: track 5.77 -> 45.8 mm, vias 2 -> 3
- net /TX1: track 44.2 -> 32.8 mm
- net GND: track 283.1 -> 289.3 mm
- net /VCCCPU: track 165.7 -> 160.5 mm
- net /CANRX: track 5.91 -> 6.86 mm
- net /RF2MOSI: track 3.61 -> 4.50 mm
- net /A2: track 16.2 -> 15.5 mm
- net Net-(D2-Pad2): track 1.43 -> 2.14 mm
- net /GPSRX: track 18.2 -> 18.7 mm
- net /GPSTX: track 19.2 -> 19.8 mm
